File: pcb/case_controller/case_controller.kicad_pcb (KiCad board)
At the start: 2 copper layers, 81.3 x 63.5 mm, 8 parts

Commit message: Update TODO
Other:
- board text removed: "TODO: Bodge/Voltage Dividers?"
Changed lines of the file:
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@@
-    (effects (font (size 1 1) (thickness 0.15)) (justify left bottom))
-  )
-  (gr_text "TODO: Bodge/Voltage Dividers?" (at 132.08 58.42) (layer "F.SilkS")
     (effects (font (size 1 1) (thickness 0.15)) (justify left bottom))
   )
